File: kicad/IO_Bed.kicad_sch (KiCad schematic)
At the start: 43 parts, among them J3 DIN-7, J4 DIN-7, J5 SJ1-3533NG, J6 SJ1-3533NG, J7 SJ1-3533NG, U10 CPC1017N, U2 MCP23017_SS, U3 CPC1017N, U4 CPC1017N, U5 CPC1017N, U6 CPC1017N, U7 CPC1017N, U8 CPC1017N, U9 CPC1017N

Commit message: Small updates/descriptions
Other:
- note added: "FROM HANDSET"
- note added: "TO BED"
Changed lines of the file:
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@@
     (stroke (width 0) (type default) (color 0 0 0 0))
+  )
+  (text "TO BED" (at 237.49 35.56 0)
+    (effects (font (size 4 4)) (justify left bottom))
+  )
+  (text "FROM HANDSET" (at 219.71 139.7 0)
+    (effects (font (size 4 4)) (justify left bottom))
   )
   (label "DIN_IN_COMMON" (at 181.61 129.54 0)

Commit message: updated design
Parts:
- C10, C11, C12, C13, C14, C15, C16, C17, C18, C8, C9: value 100nF 0805 -> 100nF 0603; EuroCircuits (none) -> GPC0603104; JLCPCB (none) -> CC0603KRX7R9BB104; LCSC (none) -> C14663
- J3, J4: EuroCircuits (none) -> PSG03465
- J5, J6, J7: EuroCircuits (none) -> SJ1-3533NG
- JP1: footprint Connector_PinHeader_2.54mm:PinHeader_1x03_P2.54mm_Vertical_SMD_Pin1Left -> Connector_PinHeader_2.54mm:PinHeader_1x03_P2.54mm_Vertical; EuroCircuits (none) -> M20-8770342
- R10, R11, R12: EuroCircuits (none) -> GPR080510K; JLCPCB (none) -> 0805W8F1002T5E; LCSC (none) -> C17414
- R13, R15: EuroCircuits (none) -> GPR08051M; JLCPCB (none) -> 0805W8F1004T5E; LCSC (none) -> C17514
- R14: EuroCircuits (none) -> GPR08055R6; JLCPCB (none) -> 0805W8J056JT5E; LCSC (none) -> C25321
- RN1, RN2, RN3, RN4: EuroCircuits (none) -> EXBV8V103JV; JLCPCB (none) -> 4D03WGF1002T5(E); LCSC (none) -> C109324
- RN5, RN6: value 270 -> 1.5k; EuroCircuits (none) -> EXB-38V152JV; JLCPCB (none) -> 4D03WGJ0152T5E; LCSC (none) -> C11988
- RN7, RN8: value 1k -> 1.5k; EuroCircuits (none) -> EXB-38V152JV; JLCPCB (none) -> 4D03WGJ0152T5E; LCSC (none) -> C11988
- TP6, TP7, TP8: EuroCircuits (none) -> 5006
- U10, U3, U4, U5, U6, U7, U8, U9: EuroCircuits (none) -> CPC1017NTR; JLCPCB (none) -> CPC1017NTR; LCSC (none) -> C81521
- U2: value MCP23017_SS -> MCP23017-E/SO; EuroCircuits (none) -> MCP23017-E/SO; JLCPCB (none) -> MCP23017-E/SO
Connections:
- net ~{RESET}: now reaches R12.2, U2.18 (~{RESET})

Commit message: BOM changes; RPi thermal gap
Parts:
- J3, J4: DNS (none) -> X; MPN (none) -> PSG03465
- J5, J6, J7: DNS (none) -> X; MPN (none) -> SJ1-3533NG
- JP1: MPN (none) -> M20-8770342
- R10, R11, R12: value 10k -> 10k 0805
- R13, R15: value 1M -> 1M 0805
- R14: value 5.6 -> 5.6 0805
- RN1, RN2, RN3, RN4: value 10k -> 10k 4x0603; MPN (none) -> EXBV8V103JV
- RN5, RN6, RN7, RN8: value 1.5k -> 1.5k 4x0603; MPN (none) -> EXB-38V152JV
- TP6, TP7, TP8: value TestPoint -> KeyStone 5006; DNS (none) -> X; MPN (none) -> 5006
- U10, U3, U4, U5, U6, U7, U8, U9: MPN (none) -> CPC1017NTR
- U2: MPN (none) -> MCP23017-E/SO

Commit message: start changing relays
Parts:
- removed JP1: Jumper, Connector_PinHeader_2.54mm:PinHeader_1x03_P2.54mm_Vertical, symbol Jumper:Jumper_3_Bridged12
- removed TP6: KeyStone 5006, TestPoint:TestPoint_Keystone_5005-5009_Compact, symbol Connector:TestPoint
- removed U3, U4, U5, U6, U7, U8: CPC1017N, Package_SO:SOP-4_3.8x4.1mm_P2.54mm, symbol Relay_SolidState:CPC1017N
- added D4: (no value), symbol Diode:B160-E3
- added D5, D6, D7, D8, D9: B160-E3, Diode_SMD:D_SMA, symbol Diode:B160-E3
- added F3: (no value), symbol Device:Polyfuse
- added K1: (no value), symbol Relay:G5Q-1A
- added K2, K3, K4, K5, K6: G5Q-1A, Relay_THT:Relay_SPST_Omron-G5Q-1A, symbol Relay:G5Q-1A
- added Q4: (no value), symbol Transistor_FET:2N7002E
- added Q5, Q6, Q7, Q8, Q9: 2N7002E, Package_TO_SOT_SMD:SOT-23, symbol Transistor_FET:2N7002E
- TP7, TP8: value KeyStone 5006 -> (none); footprint TestPoint:TestPoint_Keystone_5005-5009_Compact -> (none)
Connections:
- net +3V3: no longer RN2.5 (R4.2), RN2.6 (R3.2), RN2.7 (R2.2), RN2.8 (R1.2), RN3.5 (R4.2), RN3.6 (R3.2), RN3.7 (R2.2), RN3.8 (R1.2), U10.1, U9.1
- net +5V: now also R14.2, U10.1, U9.1, D4.1 (K), D5.1 (K), D6.1 (K), D7.1 (K), D8.1 (K), D9.1 (K), K1.5, K2.5, K3.5, K4.5, K5.5, K6.5
- net DIN_OUT_COMMON: now also TP7.1, F3.1, K1.3, K2.3, K3.3, K4.3, K5.3, K6.3; no longer J4.1
- net GND: now also Q4.2 (S), Q5.2 (S), Q6.2 (S), Q7.2 (S), Q8.2 (S), Q9.2 (S)
- net CTL_M1_DN: now reaches RN5.6 (R3.2)
- net CTL_M1_DN: now also Q5.1 (G)
- net M2_UP: now reaches J4.3
- net M2_UP: now also K3.2
- net at RN2.1 (R1.1), RN5.1 (R1.1): no longer U2.4 (GPB3)
- net at RN2.2 (R2.1), RN5.2 (R2.1): no longer U2.3 (GPB2)
- net at RN2.3 (R3.1), RN5.3 (R3.1): no longer U2.2 (GPB1)
- net at RN2.4 (R4.1), RN5.4 (R4.1): no longer U2.1 (GPB0)
- net CTL_M1_UP: now reaches RN5.5 (R4.2)
- net CTL_M1_UP: now also Q4.1 (G)
- net CTL_M2_UP: now reaches RN5.7 (R2.2)
- net CTL_M2_UP: now also Q6.1 (G)
- net CTL_M2_DN: now reaches RN5.8 (R1.2)
- net CTL_M2_DN: now also Q7.1 (G)
- net CTL_EX1: now reaches RN6.7 (R2.2), U9.2
- net at RN3.1 (R1.1), RN6.1 (R1.1): no longer U2.8 (GPB7)
- net at RN3.2 (R2.1), RN6.2 (R2.1): no longer U2.7 (GPB6)
- net at RN3.3 (R3.1), RN6.3 (R3.1): no longer U2.6 (GPB5)
- net at RN3.4 (R4.1), RN6.4 (R4.1): no longer U2.5 (GPB4)
- net CTL_M3_UP: now reaches RN6.5 (R4.2)
- net CTL_M3_UP: now also Q8.1 (G)
- net CTL_M3_DN: now reaches RN6.6 (R3.2)
- net CTL_M3_DN: now also Q9.1 (G)
- net CTL_EX2: now reaches RN6.8 (R1.2), U10.2
- net M3_DN: now reaches J4.7
- net M3_DN: now also K6.2
- net M2_DN: now reaches J4.5
- net M2_DN: now also K4.2
- net M3_UP: now reaches J4.6
- net M3_UP: now also K5.2
- net M1_DN: now reaches J4.4
- net M1_DN: now also K2.2
- net M1_UP: now reaches J4.2
- net M1_UP: now also K1.2; no longer TP7.1
- net I2C_SCL_3V3 renamed I2C_SCL_5V
- net I2C_SDA_3V3 renamed I2C_SDA_5V
- new net: D9.2 (A), K6.1, Q9.3 (D)
- new net: D5.2 (A), K2.1, Q5.3 (D)
- new net: D7.2 (A), K4.1, Q7.3 (D)
- new net: D4.2 (A), K1.1, Q4.3 (D)
- new net: RN2.5 (R4.2), RN2.6 (R3.2), RN2.7 (R2.2), RN2.8 (R1.2), RN3.5 (R4.2), RN3.6 (R3.2), RN3.7 (R2.2), RN3.8 (R1.2)
- new net: D8.2 (A), K5.1, Q8.3 (D)
- new net: D6.2 (A), K3.1, Q6.3 (D)
- new net: F3.2, J4.1
Other:
- moved on the sheet: C17, C18, J4, J7, R13, R15, RN2, RN3, RN5, RN6, RN7, TP7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
